File: boards/schematic.sch (EAGLE design)
At the start: 106 parts, among them IC1 74LS165D, J1 AVR_SPI_PRG_6NS, Q1 MOSFET-NCHANNELBSS123LT1G, U1 SD_CARD_SOCKET, U2 SD_CARD_SOCKET, U3 LCD-16X2SILK, U4 MAX1555

Commit message: Improvements to the enclosure, tweaking the PCB
Parts:
- added C28, C29: 47pf, SparkFun-Passives:CAP0603-CAP
- added C3, C30: .1uF, SparkFun-Passives:CAP0603-CAP
- added C31: 4.7uF, SparkFun-Passives:CAP0603-CAP
- added JP4: USB_MICROB_PLUGCONN-11752, SparkFun-Connectors:USB_MICROB_PLUGCONN-11752
- added R44, R45: 22, SparkFun-Passives:RESISTOR0603-RES
- added U6: FTS31XS-U, SparkFun-DigitalIC:FT231XS
Connections:
- new net +5V: C30.1, C31.1, JP4.VCC, U6.VCC
- new net N$22: C28.1, JP4.D+, R44.2
- new net N$23: C29.1, JP4.D-, R45.2
- new net N$37: R44.1, U6.USBDP
- new net N$38: R45.1, U6.USBDM
- new net N$40: C3.1, U6.!RESET, U6.3V3OUT, U6.VCCIO
- new net POS_RX_LOGIC: U6.TXD
- new net POS_TX_LOGIC: U6.RXD
- net GND: now also C28.2, C29.2, C3.2, C30.2, C31.2, JP4.GND, U1.SH@1, U1.SH@2, U2.SH@1, U2.SH@2, U6.GND@16, U6.GND@6
Changed lines of the file:
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@@
 <part name="GND51" library="supply1" deviceset="GND" device=""/>
 <part name="R43" library="SparkFun-Passives" deviceset="RESISTOR" device="0603-RES" value="1k"/>
+<part name="U6" library="SparkFun-DigitalIC" deviceset="FT231X" device="S" value="FTS31XS-U"/>
+<part name="JP4" library="SparkFun-Connectors" deviceset="USB_MICROB_PLUG" device="CONN-11752"/>
+<part name="GND2" library="supply1" deviceset="GND" device=""/>
+<part name="P+14" library="supply1" deviceset="+5V" device=""/>
+<part name="P+15" library="supply1" deviceset="+5V" device=""/>
+<part name="GND52" library="supply1" deviceset="GND" device=""/>
+<part name="R44" library="SparkFun-Passives" deviceset="RESISTOR" device="0603-RES" value="22"/>
+<part name="R45" library="SparkFun-Passives" deviceset="RESISTOR" device="0603-RES" value="22"/>
+<part name="C3" library="SparkFun-Passives" deviceset="CAP" device="0603-CAP" value=".1uF"/>
+<part name="C28" library="SparkFun-Passives" deviceset="CAP" device="0603-CAP" value="47pf"/>
+<part name="C29" library="SparkFun-Passives" deviceset="CAP" device="0603-CAP" value="47pf"/>
+<part name="GND53" library="supply1" deviceset="GND" device=""/>
+<part name="GND54" library="supply1" deviceset="GND" device=""/>
+<part name="C30" library="SparkFun-Passives" deviceset="CAP" device="0603-CAP" value=".1uF"/>
+<part name="C31" library="SparkFun-Passives" deviceset="CAP" device="0603-CAP" value="4.7uF"/>
+<part name="GND55" library="supply1" deviceset="GND" device=""/>
+<part name="GND56" library="supply1" deviceset="GND" device=""/>
+<part name="P+16" library="supply1" deviceset="+5V" device=""/>
+<part name="P+17" library="supply1" deviceset="+5V" device=""/>
 </parts>
 <sheets>
@@
 <instance part="GND51" gate="1" x="149.86" y="12.7"/>
 <instance part="R43" gate="G$1" x="132.08" y="20.32"/>
+<instance part="U6" gate="G$1" x="167.64" y="-45.72"/>
+<instance part="JP4" gate="G$1" x="114.3" y="-35.56" rot="R180"/>
+<instance part="GND2" gate="1" x="149.86" y="-76.2"/>
+<instance part="P+14" gate="1" x="149.86" y="-25.4"/>
+<instance part="P+15" gate="1" x="124.46" y="-43.18" rot="R180"/>
+<instance part="GND52" gate="1" x="127" y="-27.94" rot="R180"/>
+<instance part="R44" gate="G$1" x="139.7" y="-35.56" rot="R180"/>
+<instance part="R45" gate="G$1" x="139.7" y="-38.1" rot="R180"/>
+<instance part="C3" gate="G$1" x="149.86" y="-71.12"/>
+<instance part="C28" gate="G$1" x="134.62" y="-40.64"/>
+<instance part="C29" gate="G$1" x="129.54" y="-43.18"/>
+<instance part="GND53" gate="1" x="134.62" y="-45.72"/>
+<instance part="GND54" gate="1" x="129.54" y="-48.26"/>
+<instance part="C30" gate="G$1" x="124.46" y="-66.04"/>
+<instance part="C31" gate="G$1" x="132.08" y="-66.04"/>
+<instance part="GND55" gate="1" x="132.08" y="-71.12"/>
+<instance part="GND56" gate="1" x="124.46" y="-71.12"/>
+<instance part="P+16" gate="1" x="124.46" y="-58.42"/>
+<instance part="P+17" gate="1" x="132.08" y="-58.42"/>
 </instances>
 <busses>
@@
 <wire x1="215.9" y1="38.1" x2="215.9" y2="40.64" width="0.1524" layer="91"/>
 <junction x="215.9" y="40.64"/>
+<pinref part="U1" gate="G$1" pin="SH@2"/>
+<wire x1="215.9" y1="38.1" x2="215.9" y2="35.56" width="0.1524" layer="91"/>
+<pinref part="U1" gate="G$1" pin="SH@1"/>
+<wire x1="215.9" y1="35.56" x2="215.9" y2="33.02" width="0.1524" layer="91"/>
+<junction x="215.9" y="38.1"/>
+<junction x="215.9" y="35.56"/>
 </segment>
 <segment>
@@
 <pinref part="U2" gate="G$1" pin="VSS1"/>
 <pinref part="U2" gate="G$1" pin="VSS2"/>
+<pinref part="U2" gate="G$1" pin="SH@2"/>
+<wire x1="264.16" y1="38.1" x2="264.16" y2="35.56" width="0.1524" layer="91"/>
+<pinref part="U2" gate="G$1" pin="SH@1"/>
+<wire x1="264.16" y1="35.56" x2="264.16" y2="33.02" width="0.1524" layer="91"/>
+<junction x="264.16" y="38.1"/>
+<junction x="264.16" y="35.56"/>
 </segment>
 <segment>
@@
 <pinref part="Q1" gate="G$1" pin="S"/>
 <pinref part="GND51" gate="1" pin="GND"/>
+</segment>
+<segment>
+<pinref part="JP4" gate="G$1" pin="GND"/>
+<pinref part="GND52" gate="1" pin="GND"/>
+<wire x1="121.92" y1="-30.48" x2="127" y2="-30.48" width="0.1524" layer="91"/>
+</segment>
+<segment>
+<pinref part="GND2" gate="1" pin="GND"/>
+<pinref part="C3" gate="G$1" pin="2"/>
+<pinref part="U6" gate="G$1" pin="GND@6"/>
+<pinref part="U6" gate="G$1" pin="GND@16"/>
+<wire x1="154.94" y1="-58.42" x2="154.94" y2="-60.96" width="0.1524" layer="91"/>
+<wire x1="154.94" y1="-60.96" x2="154.94" y2="-73.66" width="0.1524" layer="91"/>
+<junction x="154.94" y="-60.96"/>
+<wire x1="154.94" y1="-73.66" x2="149.86" y2="-73.66" width="0.1524" layer="91"/>
+<junction x="149.86" y="-73.66"/>
+</segment>
+<segment>
+<pinref part="C28" gate="G$1" pin="2"/>
+<pinref part="GND53" gate="1" pin="GND"/>
+</segment>
+<segment>
+<pinref part="C29" gate="G$1" pin="2"/>
+<pinref part="GND54" gate="1" pin="GND"/>
+</segment>
+<segment>
+<pinref part="C31" gate="G$1" pin="2"/>
+<pinref part="GND55" gate="1" pin="GND"/>
+</segment>
+<segment>
+<pinref part="C30" gate="G$1" pin="2"/>
+<pinref part="GND56" gate="1" pin="GND"/>
 </segment>
 </net>
@@
 </segment>
 </net>
+<net name="POS_TX_LOGIC" class="0">
+<segment>
+<pinref part="U6" gate="G$1" pin="RXD"/>
+<wire x1="180.34" y1="-33.02" x2="195.58" y2="-33.02" width="0.1524" layer="91"/>
+<label x="182.88" y="-33.02" size="1.778" layer="95"/>
+</segment>
+</net>
+<net name="+5V" class="0">
+<segment>
+<pinref part="JP4" gate="G$1" pin="VCC"/>
+<pinref part="P+15" gate="1" pin="+5V"/>
+<wire x1="124.46" y1="-40.64" x2="121.92" y2="-40.64" width="0.1524" layer="91"/>
+</segment>
+<segment>
+<pinref part="P+14" gate="1" pin="+5V"/>
+<pinref part="U6" gate="G$1" pin="VCC"/>
+<wire x1="149.86" y1="-27.94" x2="154.94" y2="-27.94" width="0.1524" layer="91"/>
+<wire x1="154.94" y1="-27.94" x2="154.94" y2="-30.48" width="0.1524" layer="91"/>
+</segment>
+<segment>
+<pinref part="C30" gate="G$1" pin="1"/>
+<pinref part="P+16" gate="1" pin="+5V"/>
+</segment>
+<segment>
+<pinref part="C31" gate="G$1" pin="1"/>
+<pinref part="P+17" gate="1" pin="+5V"/>
+</segment>
+</net>
+<net name="POS_RX_LOGIC" class="0">
+<segment>
+<pinref part="U6" gate="G$1" pin="TXD"/>
+<wire x1="180.34" y1="-30.48" x2="195.58" y2="-30.48" width="0.1524" layer="91"/>
+<label x="182.88" y="-30.48" size="1.778" layer="95"/>
+</segment>
+</net>
+<net name="N$22" class="0">
+<segment>
+<pinref part="JP4" gate="G$1" pin="D+"/>
+<pinref part="R44" gate="G$1" pin="2"/>
+<wire x1="121.92" y1="-35.56" x2="134.62" y2="-35.56" width="0.1524" layer="91"/>
+<pinref part="C28" gate="G$1" pin="1"/>
+<junction x="134.62" y="-35.56"/>
+</segment>
+</net>
+<net name="N$23" class="0">
+<segment>
+<pinref part="JP4" gate="G$1" pin="D-"/>
+<pinref part="R45" gate="G$1" pin="2"/>
+<wire x1="121.92" y1="-38.1" x2="129.54" y2="-38.1" width="0.1524" layer="91"/>
+<pinref part="C29" gate="G$1" pin="1"/>
+<wire x1="129.54" y1="-38.1" x2="134.62" y2="-38.1" width="0.1524" layer="91"/>
+<junction x="129.54" y="-38.1"/>
+</segment>
+</net>
+<net name="N$37" class="0">
+<segment>
+<pinref part="R44" gate="G$1" pin="1"/>
+<wire x1="144.78" y1="-35.56" x2="149.86" y2="-35.56" width="0.1524" layer="91"/>
+<wire x1="149.86" y1="-35.56" x2="149.86" y2="-43.18" width="0.1524" layer="91"/>
+<pinref part="U6" gate="G$1" pin="USBDP"/>
+<wire x1="149.86" y1="-43.18" x2="154.94" y2="-43.18" width="0.1524" layer="91"/>
+</segment>
+</net>
+<net name="N$38" class="0">
+<segment>
+<pinref part="R45" gate="G$1" pin="1"/>
+<pinref part="U6" gate="G$1" pin="USBDM"/>
+<wire x1="144.78" y1="-38.1" x2="154.94" y2="-38.1" width="0.1524" layer="91"/>
+<wire x1="154.94" y1="-38.1" x2="154.94" y2="-40.64" width="0.1524" layer="91"/>
+</segment>
+</net>
+<net name="N$40" class="0">
+<segment>
+<pinref part="U6" gate="G$1" pin="3V3OUT"/>
+<pinref part="U6" gate="G$1" pin="VCCIO"/>
+<wire x1="154.94" y1="-33.02" x2="154.94" y2="-35.56" width="0.1524" layer="91"/>
+<wire x1="154.94" y1="-35.56" x2="152.4" y2="-35.56" width="0.1524" layer="91"/>
+<junction x="154.94" y="-35.56"/>
+<wire x1="152.4" y1="-35.56" x2="152.4" y2="-48.26" width="0.1524" layer="91"/>
+<pinref part="U6" gate="G$1" pin="!RESET"/>
+<wire x1="152.4" y1="-48.26" x2="154.94" y2="-48.26" width="0.1524" layer="91"/>
+<pinref part="C3" gate="G$1" pin="1"/>
+<wire x1="152.4" y1="-48.26" x2="149.86" y2="-48.26" width="0.1524" layer="91"/>
+<wire x1="149.86" y1="-48.26" x2="149.86" y2="-66.04" width="0.1524" layer="91"/>
+<junction x="152.4" y="-48.26"/>
+</segment>
+</net>
